Commit message: Removed zero origin tags from dock xacro

File: ca_description/urdf/dock/dock.xacro (robot description, xacro)
@@ -5,5 +5,4 @@
     <link name='back'>
       <visual name='visual'>
-        <origin xyz="0 0 0" rpy="0 0 0" />
         <geometry>
           <box size="${width} ${width/3} ${width * 2/3}"/>
@@ -11,5 +10,4 @@
       </visual>
       <collision name='collision'>
-        <origin xyz="0 0 0" rpy="0 0 0" />
         <geometry>
           <box size="${width} ${width/3} ${width * 2/3}"/>
@@ -18,5 +16,4 @@
       <xacro:inertial_cuboid_with_pose mass="0.15" x_length="${width}"
           y_length="${width/3}" z_length="${width * 2/3}" >
-        <origin xyz="0 0 0" />
       </xacro:inertial_cuboid_with_pose>
     </link>

Commit message: removed zero rpy prop from origin on dock.xacro

File: ca_description/urdf/dock/dock.xacro (robot description, xacro)
@@ -20,5 +20,5 @@
     <link name='base'>
       <visual name='visual'>
-        <origin xyz="0 ${width/2 - width/6} ${-(width * 2/3)/2}" rpy="0 0 0" />
+        <origin xyz="0 ${width/2 - width/6} ${-(width * 2/3)/2}" />
         <geometry>
           <box size="${width} ${width} 0.01"/>
@@ -26,5 +26,5 @@
       </visual>
       <collision name='collision'>
-        <origin xyz="0 ${width/2 - width/6} ${-(width * 2/3)/2}" rpy="0 0 0" />
+        <origin xyz="0 ${width/2 - width/6} ${-(width * 2/3)/2}" />
         <geometry>
           <box size="${width} ${width} 0.01"/>
@@ -33,5 +33,5 @@
       <xacro:inertial_cuboid_with_pose mass="0.05" x_length="${width}"
           y_length="${width}" z_length="0.01" >
-        <origin xyz="0 ${width/2 - width/6} ${-(width * 2/3)/2}" rpy="0 0 0" />
+        <origin xyz="0 ${width/2 - width/6} ${-(width * 2/3)/2}" />
       </xacro:inertial_cuboid_with_pose>
     </link>
