Commit message: Battery charger plugin

File: ca_description/urdf/create_base_gazebo.xacro (robot description, xacro)
@@ -38,4 +38,6 @@
         <xyzOffsets>0 0 0</xyzOffsets>
         <rpyOffsets>0 0 0</rpyOffsets>
+      </plugin>
+      <plugin name="battery_charger_plugin" filename="libbattery_charger_plugin.so">
       </plugin>
     </gazebo>

File: ca_description/urdf/dock/dock.xacro (robot description, xacro)
@@ -16,7 +16,8 @@
       <xacro:inertial_cuboid_with_pose mass="0.15" x_length="${width}"
           y_length="${width/3}" z_length="${width * 2/3}" >
+        <origin xyz="0 0 0" />
       </xacro:inertial_cuboid_with_pose>
     </link>
-    <link name='base'>
+    <link name='link'>
       <visual name='visual'>
         <origin xyz="0 ${width/2 - width/6} ${-(width * 2/3)/2}" />
@@ -38,6 +39,9 @@
     <joint name='glue' type='fixed'>
       <parent link="back" />
-      <child link="base" />
+      <child link="link" />
     </joint>
+    <!-- <gazebo>
+      <plugin name="model_pose_publisher_plugin" filename="libmodel_pose_publisher_plugin.so"/>
+    </gazebo> -->
   </xacro:macro>
   <xacro:dock width="0.15">
