Commit message: Add battery plugin using brass_gazebo_battery (#241)
* Add plugin usign brass_gazebo_battery

* Fix typo in static test

* Decrease RTF of the static test

* Revert static test

* Add brass_gazebo_battery as dependency

* Improve instability tweaking link

File: ca_description/urdf/create_base.xacro (robot description, xacro)
@@ -75,7 +75,11 @@
       <origin xyz="0.13 0 ${caster_z}"/>
     </xacro:caster_wheel>
-    <xacro:battery>
+    <xacro:battery_sensor
+        voltage="14.4"
+        capacity_ah="4.5"
+        charge_current="0.2"
+        discharge_current="1.9">
       <origin xyz="0.085 0 ${base_height}"/>
-    </xacro:battery>
+    </xacro:battery_sensor>
     <!-- Simulation sensors -->
     <xacro:sim_create_base/>

File: ca_description/urdf/create_battery.xacro (robot description, xacro)
@@ -1,9 +1,13 @@
 <?xml version="1.0" ?>
 <robot xmlns:xacro="http://ros.org/wiki/xacro">
-<xacro:macro name="battery" params="name:=battery parent:=base_footprint *origin">
+<xacro:macro name="battery_sensor"
+             params="name:=battery parent:=base_footprint
+                     voltage capacity_ah charge_current discharge_current
+                     *origin">
   <xacro:include filename="$(find ca_description)/urdf/utils/inertias.xacro"/>
   <xacro:include filename="$(find ca_description)/urdf/utils/conversions.xacro"/>
   <xacro:property name="parent_link" value="${parent}"/>
   <xacro:property name="link_name"   value="${name}_link"/>
+  <xacro:property name="dummy_link"  value="${link_name}_dummy"/>
   <xacro:property name="mass"        value="1"/>
   <xacro:property name="size_x_in"   value="2.2"/>
@@ -26,7 +30,40 @@
     </visual>
   </link>
+  <joint name="${name}_dummy_joint" type="continuous">
+    <parent link="${parent_link}"/>
+    <child link="${dummy_link}"/>
+    <!-- <limit effort="10" velocity="10" /> -->
+    <!-- <dynamics damping="0.1" friction="1000.0"/> -->
+  </joint>
+  <link name="${dummy_link}">
+    <xacro:dummy_inertia/>
+  </link>
   <gazebo reference="${link_name}">
     <material>Gazebo/ZincYellow</material>
   </gazebo>
+  <gazebo reference="${dummy_link}">
+    <battery name="${name}">
+      <voltage>${voltage}</voltage>
+    </battery>
+  </gazebo>
+  <gazebo>
+    <plugin name="battery_discharge" filename="libbattery_discharge.so">
+      <ros_node>${name}</ros_node>
+      <link_name>${dummy_link}</link_name>
+      <battery_name>${name}</battery_name>
+      <constant_coef>${voltage}</constant_coef>
+      <linear_coef>${-voltage/4}</linear_coef>
+      <initial_charge>${capacity_ah}</initial_charge>
+      <capacity>${capacity_ah}</capacity>
+      <resistance>0.061523</resistance>
+      <smooth_current_tau>1.9499</smooth_current_tau>
+      <charge_rate>${charge_current}</charge_rate>
+    </plugin>
+    <plugin name="battery_consumer" filename="libbattery_consumer.so">
+      <link_name>${dummy_link}</link_name>
+      <battery_name>${name}</battery_name>
+      <power_load>${discharge_current * voltage}</power_load>
+    </plugin>
+  </gazebo>
 </xacro:macro>
 </robot>

Commit message: Add robot + battery namespace (#243)

File: ca_description/urdf/create_base.xacro (robot description, xacro)
@@ -76,4 +76,5 @@
     </xacro:caster_wheel>
     <xacro:battery_sensor
+        namespace="${robot_name}"
         voltage="14.4"
         capacity_ah="4.5"

File: ca_description/urdf/create_battery.xacro (robot description, xacro)
@@ -2,5 +2,5 @@
 <robot xmlns:xacro="http://ros.org/wiki/xacro">
 <xacro:macro name="battery_sensor"
-             params="name:=battery parent:=base_footprint
+             params="name:=battery parent:=base_footprint namespace:=create
                      voltage capacity_ah charge_current discharge_current
                      *origin">
@@ -33,6 +33,4 @@
     <parent link="${parent_link}"/>
     <child link="${dummy_link}"/>
-    <!-- <limit effort="10" velocity="10" /> -->
-    <!-- <dynamics damping="0.1" friction="1000.0"/> -->
   </joint>
   <link name="${dummy_link}">
@@ -49,5 +47,5 @@
   <gazebo>
     <plugin name="battery_discharge" filename="libbattery_discharge.so">
-      <ros_node>${name}</ros_node>
+      <ros_node>${namespace}</ros_node>
       <link_name>${dummy_link}</link_name>
       <battery_name>${name}</battery_name>
